File: ElectronicDesignAutomation/WifiSwitch.sch (KiCad schematic (older format))
At the start: 9 parts, among them P1 CONN_01X05, P2 CONN_01X03, U1 ESP8266_ESP3, U2 MOC3031S, U3 TRIAC

Commit message: Updated Schematic
Updates Schematic and added PCB design
Parts:
- R2: value 10K -> 4K7
Connections:
- net +3V3: now also U1.13 (GPIO2)
- net at R2.1, U1.6 (CH_PD): no longer U1.13 (GPIO2)
Changed lines of the file:
@@
-$EndComp
-$Comp
-L AC_to_DC_convertor C1
-U 1 1 5537CAC0
-P 6950 4200
-F 0 "C1" H 7050 4100 60  0000 C CNN
-F 1 "AC_to_DC_convertor" H 6950 4450 60  0000 C CNN
-F 2 "WifiSwitch:AC_DC_Conv" H 7050 4200 60  0001 C CNN
-F 3 "" H 7050 4200 60  0000 C CNN
-	1    6950 4200
-	1    0    0    -1
 $EndComp
 $Comp
@@
 P 5500 3650
 F 0 "R2" V 5580 3650 50  0000 C CNN
-F 1 "10K" V 5500 3650 50  0000 C CNN
+F 1 "4K7" V 5500 3650 50  0000 C CNN
 F 2 "Resistors_SMD:R_1206_HandSoldering" V 5430 3650 30  0001 C CNN
 F 3 "" H 5500 3650 30  0000 C CNN
@@
 Connection ~ 3500 5250
 Wire Wire Line
-	4950 3450 4800 3450
+	4800 3450 5500 3450
 Wire Wire Line
 	6900 2350 6900 1900
@@
 	6100 3450 6100 3600
 Connection ~ 6900 3600
-Wire Wire Line
-	6100 3150 6100 2800
-Wire Wire Line
-	6100 2800 5800 2800
 Wire Wire Line
 	6400 2950 6100 2950
@@
 	3700 3850 3750 3850
 Wire Wire Line
-	3700 3050 3700 3850
-Wire Wire Line
-	3700 3050 5500 3050
-Wire Wire Line
 	3600 3350 3600 4550
 Wire Wire Line
@@
 Wire Wire Line
 	4800 3950 5200 3950
-Wire Wire Line
-	5500 3050 5500 3500
-Wire Wire Line
-	4950 3450 4950 3050
-Connection ~ 4950 3050
 Wire Wire Line
 	5500 3800 5500 4100
@@
 	6100 4000 6100 4100
 Connection ~ 6100 4100
+Wire Wire Line
+	6100 2800 6100 3150
+Wire Wire Line
+	6100 2800 5800 2800
+Wire Wire Line
+	3700 3850 3700 3350
+Connection ~ 3700 3350
+Wire Wire Line
+	5500 3450 5500 3500
+$Comp
+L AC_to_DC_convertor C1
+U 1 1 5537CAC0
+P 6950 4200
+F 0 "C1" H 7050 4100 60  0000 C CNN
+F 1 "AC_to_DC_convertor" H 6950 4450 60  0000 C CNN
+F 2 "WifiSwitch:AC_DC_Conv" H 7050 4200 60  0001 C CNN
+F 3 "" H 7050 4200 60  0000 C CNN
+	1    6950 4200
+	1    0    0    -1
+$EndComp
 $EndSCHEMATC
